File: PCB_Kicad/PCB/project233/project233.kicad_sch (KiCad schematic)
At the start: 0 parts

Commit message: update Kicad PCB
Other:
- added sheet POWER (POWER.kicad_sch)
Changed lines of the file:
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@@
 (kicad_sch (version 20230121) (generator eeschema)
   (paper "A4")
-  (sheet (at 108.966 72.39) (size 40.386 50.292) (fields_autoplaced)
+  (sheet (at 122.428 73.66) (size 40.386 50.292) (fields_autoplaced)
     (stroke (width 0.1524) (type solid))
     (fill (color 0 0 0 0.0000))
-    (property "Sheetname" "MCU" (at 108.966 71.6784 0)
+    (property "Sheetname" "MCU" (at 122.428 72.9484 0)
       (effects (font (size 1.27 1.27)) (justify left bottom))
     )
-    (property "Sheetfile" "MCU.kicad_sch" (at 108.966 123.2666 0)
+    (property "Sheetfile" "MCU.kicad_sch" (at 122.428 124.5366 0)
       (effects (font (size 1.27 1.27)) (justify left top))
     )
@@
     )
   )
-  (sheet (at 169.672 84.582) (size 38.1 26.416) (fields_autoplaced)
+  (sheet (at 183.134 85.852) (size 38.1 26.416) (fields_autoplaced)
     (stroke (width 0.1524) (type solid))
     (fill (color 0 0 0 0.0000))
-    (property "Sheetname" "SENS" (at 169.672 83.8704 0)
+    (property "Sheetname" "SENS" (at 183.134 85.1404 0)
       (effects (font (size 1.27 1.27)) (justify left bottom))
     )
-    (property "Sheetfile" "SENS.kicad_sch" (at 169.672 111.5826 0)
+    (property "Sheetfile" "SENS.kicad_sch" (at 183.134 112.8526 0)
       (effects (font (size 1.27 1.27)) (justify left top))
     )
@@
       )
     )
+  )
+  (sheet (at 59.436 86.614) (size 33.02 28.702) (fields_autoplaced)
+    (stroke (width 0.1524) (type solid))
+    (fill (color 0 0 0 0.0000))
+    (property "Sheetname" "POWER" (at 59.436 85.9024 0)
+      (effects (font (size 1.27 1.27)) (justify left bottom))
+    )
+    (property "Sheetfile" "POWER.kicad_sch" (at 59.436 115.9006 0)
+      (effects (font (size 1.27 1.27)) (justify left top))
+    )
+    (instances
+      (project "project233"
+        (path "/a9a55588-2187-4bc3-b43e-c4b5b08bd1ab" (page "4"))
+      )
+    )
