File: PCB_Kicad/PCB/project233/project233.kicad_pcb (KiCad board)
At the start: 2 copper layers, 93 x 75 mm, 63 parts, among them J1 USB_B_Micro, J2 Header_1x4, J3 Header_1x4, J4 Header_1x3, J5 Header_1x4, Q1 2SC1815, SW1 RESET, SW2 BT1, SW3 BT2, U1 STM32F103C8T6, U2 MAX30102EFD_, U3 RT9193-33GB, U4 AMS1117-1.8, U5 Batt_Holder

Commit message: update Kicad PCB
Parts:
- moved R6 3.66 mm to (135.6, 98.0)
- moved R7 2.85 mm to (133.9, 96.1), turned to 180 degrees
- moved R8 2.64 mm to (134.4, 100.6), turned to 90 degrees
- moved R5 0.64 mm to (186.2, 118.7)
- moved C12 0.50 mm to (200.7, 115.6)
- moved D4 0.25 mm to (186.2, 120.7)
Connections:
- R8 pad 2: +1V8 -> VCC
- U2 pad 10: +1V8 -> VCC
- U2 pad 9: +1V8 -> VCC
Routing:
- net GND: track 8.92 -> 279.8 mm, vias 0 -> 43
- net VCC: track 240.1 -> 271.1 mm, vias 4 -> 6
- net SCL: track 60.2 -> 65.7 mm
- net +1V8: track 78.9 -> 75.2 mm
- net SDA: track 53.0 -> 51.3 mm
- net Net-(D5-K): track 21.6 -> 22.6 mm
- added copper zone on B.Cu, net GND
- added copper zone on F.Cu, net GND

Commit message: update Kicad PCB
Parts:
- moved R8 15.9 mm to (119.1, 105.2), turned to -90 degrees
- moved J5 13.0 mm to (155.7, 84.1)
- moved R6 11.6 mm to (124.2, 99.8), turned to 0 degrees
- moved C3 10.5 mm to (152.7, 102.9)
- moved R1 10.5 mm to (149.9, 100.3)
- moved SW1 10.4 mm to (155.7, 99.8)
- moved R7 9.44 mm to (129.3, 104.4), turned to 90 degrees
- moved U2 8.50 mm to (123.3, 103.9)
- moved G*** 8.34 mm to (135.4, 104.4)
- moved C20 7.61 mm to (124.0, 108.3), turned to -90 degrees
- moved BZ1 7.22 mm to (130.8, 117.9)
- moved Q1 7.01 mm to (138.9, 117.3)
- moved R10 6.77 mm to (142.2, 117.3), turned to 90 degrees
- moved C19 4.37 mm to (126.2, 108.3), turned to -90 degrees
Routing:
- net GND: track 279.8 -> 260.8 mm, vias 43 -> 41
- net SDA: track 51.3 -> 62.9 mm
- net VCC: track 271.1 -> 280.8 mm
- net /MCU/BUZZER_EN: track 35.0 -> 41.0 mm
- net Net-(U2-~{INT}): track 3.13 -> 6.38 mm
- net +1V8: track 75.2 -> 78.3 mm
- net SCL: track 65.7 -> 64.7 mm
- net /MCU/USB-: track 22.1 -> 21.3 mm
- net /MCU/NRST: track 28.5 -> 29.4 mm
- net /MCU/BT_2: track 28.8 -> 29.6 mm
- net /MCU/BT_1: track 42.8 -> 42.1 mm
Other:
- board text added: "RESET"

Commit message: export Gerber
Parts:
- moved R2 1.44 mm to (167.2, 90.2)
- moved G*** 1.02 mm to (135.5, 105.4)
- moved C7 1.02 mm to (171.4, 89.4)
Routing:
- net GND: track 260.8 -> 330.7 mm, vias 41 -> 52
- net VCC: track 280.8 -> 283.8 mm
- net Net-(D1-K): track 1.99 -> 3.43 mm
- net /MCU/DEBUG_LED: track 8.11 -> 6.91 mm
