File: PCB_Kicad/PCB/project233/project233.kicad_pcb (KiCad board)
At the start: 2 copper layers, 93 x 75 mm, 63 parts, among them J1 USB_B_Micro, J2 Header_1x4, J3 Header_1x4, J4 Header_1x3, J5 Header_1x4, Q1 2SC1815, SW1 RESET, SW2 BT1, SW3 BT2, U1 STM32F103C8T6, U2 MAX30102EFD_, U3 RT9193-33GB, U4 AMS1117-1.8, U5 Batt_Holder

Commit message: update KICAD PCB
Parts:
- moved G*** 0.77 mm to (135.6, 104.6)
Connections:
- R8 pad 1: Net-(U2-~{INT}) -> ~INT
- U1 pad 12: unconnected-(U1-PA2-Pad12) -> ~INT
- U2 pad 13: Net-(U2-~{INT}) -> ~INT
Routing:
- net ~INT: track 0.00 -> 68.5 mm, vias 0 -> 2
- net GND: track 330.7 -> 371.5 mm, vias 52 -> 55
- net Net-(U2-~{INT}): track 6.38 -> 0.00 mm
