File: PCB_Kicad/PCB/project233/MCU.kicad_sch (KiCad schematic)
At the start: 21 parts, among them J2 USB_B_Micro, SW1 RESET, U1 STM32F103C8T6

Commit message: update Kicad PCB
Parts:
- removed SW1: RESET, Button_SMD:Button_3x6_SMD, symbol Switch:SW_Push
- added BZ1: Buzzer, Buzzer:Buzzer_9056_THT, symbol Device:Buzzer
- added C1 (x2): 100nF, Capacitor_SMD:C_0805_2012Metric, symbol Device:C
- added J1: Header_1x3, Connector_PinHeader_2.54mm:PinHeader_1x03_P2.54mm_Vertical, symbol Connector:Conn_01x03_Pin
- added J3 (x2): Header_1x4, Connector_PinHeader_2.54mm:PinHeader_1x04_P2.54mm_Vertical, symbol Connector:Conn_01x04_Pin
- added Q1: 2SC1815, Package_TO_SOT_SMD:SOT-23, symbol NPN_Trans_2SC1815:2SC1815
- added R1: 150R, Resistor_SMD:R_0603_1608Metric, symbol Device:R_Small
- added R1: 10k, Resistor_SMD:R_0603_1608Metric, symbol Device:R_Small
- added R2 (x2): 1k, Resistor_SMD:R_0603_1608Metric, symbol Device:R_Small
- added SW2: BT1, Button_SMD:Button_3x6_SMD, symbol Switch:SW_Push
- added SW2: RESET, Button_SMD:Button_3x6_SMD, symbol Switch:SW_Push
- added SW2: BT2, Button_SMD:Button_3x6_SMD, symbol Switch:SW_Push
- C1, C10, C11, C16, C2, C3, C4, C5, C6, C7, C9: footprint Capacitor_SMD:C_0402_1005Metric -> Capacitor_SMD:C_0805_2012Metric
- D3: footprint Diode_SMD:D_SOD-123 -> Diode_SMD:D_SOD-123F
- J3: value ~ -> Header_1x4; Name (none) -> SW Connector
Connections:
- net BOOT0: now also R1.2
- net GND: now also C1.2, C1.2, J1.1 (Pin_1), J3.1 (Pin_1), J3.2 (Pin_2), Q1.2 (E), SW2.2, SW2.2, SW2.2
- net NRST: now also SW2.1
- net VCC: now also BZ1.1 (-), J1.3 (Pin_3), J3.1 (Pin_1), J3.2 (Pin_2), R2.1, R2.1
- net BUZZER_EN: now reaches U1.13 (PA3)
- net BUZZER_EN: now also R1.2
- net BT_1: now reaches U1.14 (PA4)
- net BT_1: now also C1.1, R2.2, SW2.1
- net BT_2: now reaches U1.15 (PA5)
- net BT_2: now also C1.1, R2.2, SW2.1
- net RX: now reaches U1.30 (PA9)
- net RX: now also J3.3 (Pin_3)
- net TX: now reaches U1.31 (PA10)
- net TX: now also J3.4 (Pin_4)
- net LCD_SCL renamed SCL
- net SCL: now also J3.3 (Pin_3)
- net LCD_SDA renamed SDA
- net SDA: now also J3.4 (Pin_4)
- net LOAD_CTR: no longer names the net of U1.18 (PB0)
- new net: Q1.1 (B), R1.1
- new net: BZ1.2 (+), Q1.3 (C)
- new net: J1.2 (Pin_2), R1.1
- no-connect marks 22 -> 24
Other:
- moved on the sheet: C1, C10, C11, C16, C2, C3, C4, C5, C6, C7, C9, D1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

Commit message: update KICAD PCB
Connections:
- net ~INT: now reaches U1.12 (PA2)
- no-connect marks 24 -> 23
Changed lines of the file:
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@@
   (no_connect (at 120.396 82.804))
   (no_connect (at 120.396 105.664))
-  (no_connect (at 120.396 72.644))
   (no_connect (at 87.376 95.504))
   (no_connect (at 240.284 91.44))
@@
     (stroke (width 0) (type default))
   )
+  (wire (pts (xy 120.396 72.644) (xy 133.35 72.644))
+    (stroke (width 0) (type default))
+  )
   (wire (pts (xy 120.396 95.504) (xy 133.604 95.504))
     (stroke (width 0) (type default))
@@
   (label "HSE_OUT" (at 70.358 80.264 0) (fields_autoplaced)
     (effects (font (size 0.762 0.762)) (justify left bottom))
+  )
+  (label "~INT" (at 133.35 72.644 180) (fields_autoplaced)
+    (effects (font (size 1.27 1.27)) (justify right bottom))
   )
   (label "BT_1" (at 247.65 41.148 180) (fields_autoplaced)
@@
     )
   )
+  (global_label "~INT" (shape input) (at 133.35 72.644 0) (fields_autoplaced)
+    (effects (font (size 1.27 1.27)) (justify left))
+    (property "Intersheetrefs" "${INTERSHEET_REFS}" (at 140.0658 72.644 0)
+      (effects (font (size 1.27 1.27)) (justify left) hide)
+    )
+  )
