File: PCB_Kicad/PCB/project233/SENS.kicad_sch (KiCad schematic)
At the start: 0 parts

Commit message: update Kicad PCB
Parts:
- added C9: 100n, Capacitor_SMD:C_0805_2012Metric, symbol Device:C
- added C9: 10uF, Capacitor_SMD:C_0805_2012Metric, symbol Device:C
- added R1 (x3): 1K, Resistor_SMD:R_0603_1608Metric, symbol Device:R_Small
- added U2: MAX30102EFD_, MAX30102EFD_:21-1048_F143A5&plus_1_MXM, symbol MAX30102EFD_:MAX30102EFD_
Connections:
- new net: R1.1, U2.13 (~{INT})
- new net +1V8: C9.1, C9.1, R1.2, U2.10 (VLED+), U2.11 (VDD), U2.9 (VLED+)
- new net GND: C9.2, C9.2, U2.12 (GND), U2.4 (PGND)
- new net SCL: R1.2, U2.2 (SCL)
- new net SDA: R1.2, U2.3 (SDA)
- new net VCC: R1.1, R1.1
- no-connect marks 0 -> 2

Commit message: update Kicad PCB
Connections:
- net +1V8: no longer R1.2, U2.10 (VLED+), U2.9 (VLED+)
- net VCC: now also R1.2, U2.10 (VLED+), U2.9 (VLED+)
Other:
- moved on the sheet: C9
Changed lines of the file:
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@@
   (junction (at 157.988 92.964) (diameter 0) (color 0 0 0 0)
   )
-  (junction (at 180.594 84.328) (diameter 0) (color 0 0 0 0)
+  (junction (at 180.594 72.644) (diameter 0) (color 0 0 0 0)
+  )
+  (junction (at 111.252 94.488) (diameter 0) (color 0 0 0 0)
   )
   (junction (at 164.592 87.376) (diameter 0) (color 0 0 0 0)
   )
-  (junction (at 111.252 94.488) (diameter 0) (color 0 0 0 0)
-  )
   (junction (at 160.528 107.188) (diameter 0) (color 0 0 0 0)
   )
-  (junction (at 164.592 84.328) (diameter 0) (color 0 0 0 0)
-  )
-  (junction (at 168.91 84.328) (diameter 0) (color 0 0 0 0)
-  )
-  (junction (at 180.594 91.948) (diameter 0) (color 0 0 0 0)
+  (junction (at 168.91 72.644) (diameter 0) (color 0 0 0 0)
+  )
+  (junction (at 180.594 80.264) (diameter 0) (color 0 0 0 0)
   )
   (junction (at 113.792 81.788) (diameter 0) (color 0 0 0 0)
@@
     (stroke (width 0) (type default))
   )
-  (wire (pts (xy 157.988 84.328) (xy 164.592 84.328))
-    (stroke (width 0) (type default))
-  )
-  (wire (pts (xy 164.592 87.376) (xy 164.592 84.328))
-    (stroke (width 0) (type default))
-  )
   (wire (pts (xy 157.988 92.964) (xy 164.592 92.964))
     (stroke (width 0) (type default))
@@
     (stroke (width 0) (type default))
   )
+  (wire (pts (xy 164.592 85.852) (xy 164.592 87.376))
+    (stroke (width 0) (type default))
+  )
   (wire (pts (xy 163.068 87.376) (xy 164.592 87.376))
     (stroke (width 0) (type default))
@@
     (stroke (width 0) (type default))
   )
-  (wire (pts (xy 164.592 84.328) (xy 168.91 84.328))
+  (wire (pts (xy 157.988 72.644) (xy 168.91 72.644))
+    (stroke (width 0) (type default))
+  )
+  (wire (pts (xy 157.988 72.644) (xy 157.988 84.328))
     (stroke (width 0) (type default))
   )
@@
     (stroke (width 0) (type default))
   )
-  (wire (pts (xy 168.91 91.948) (xy 180.594 91.948))
+  (wire (pts (xy 168.91 80.264) (xy 180.594 80.264))
     (stroke (width 0) (type default))
   )
@@
     (stroke (width 0) (type default))
   )
-  (wire (pts (xy 168.91 84.328) (xy 180.594 84.328))
-    (stroke (width 0) (type default))
-  )
-  (wire (pts (xy 180.594 81.026) (xy 180.594 84.328))
-    (stroke (width 0) (type default))
-  )
-  (wire (pts (xy 180.594 91.948) (xy 180.594 94.742))
+  (wire (pts (xy 168.91 72.644) (xy 180.594 72.644))
+    (stroke (width 0) (type default))
+  )
+  (wire (pts (xy 180.594 69.342) (xy 180.594 72.644))
+    (stroke (width 0) (type default))
+  )
+  (wire (pts (xy 180.594 80.264) (xy 180.594 83.058))
     (stroke (width 0) (type default))
   )
@@
     )
   )
-  (symbol (lib_id "power:GND") (at 180.594 94.742 0) (unit 1)
+  (symbol (lib_id "power:GND") (at 180.594 83.058 0) (unit 1)
     (in_bom yes) (on_board yes) (dnp no)
-    (property "Reference" "#PWR024" (at 180.594 101.092 0)
-      (effects (font (size 1.27 1.27)) hide)
-    )
-    (property "Value" "GND" (at 180.594 99.06 0)
-      (effects (font (size 1.27 1.27)))
-    )
-    (property "Footprint" "" (at 180.594 94.742 0)
-      (effects (font (size 1.27 1.27)) hide)
-    )
-    (property "Datasheet" "" (at 180.594 94.742 0)
+    (property "Reference" "#PWR024" (at 180.594 89.408 0)
+      (effects (font (size 1.27 1.27)) hide)
+    )
+    (property "Value" "GND" (at 180.594 87.376 0)
+      (effects (font (size 1.27 1.27)))
+    )
+    (property "Footprint" "" (at 180.594 83.058 0)
+      (effects (font (size 1.27 1.27)) hide)
+    )
+    (property "Datasheet" "" (at 180.594 83.058 0)
       (effects (font (size 1.27 1.27)) hide)
     )
@@
     )
   )
-  (symbol (lib_id "Device:C") (at 180.594 88.138 0) (unit 1)
+  (symbol (lib_id "Device:C") (at 180.594 76.454 0) (unit 1)
     (in_bom yes) (on_board yes) (dnp no)
-    (property "Reference" "C9" (at 183.7182 86.868 0)
+    (property "Reference" "C9" (at 183.7182 75.184 0)
       (effects (font (size 1.27 1.27)) (justify left))
     )
-    (property "Value" "100n" (at 183.7182 89.408 0)
+    (property "Value" "100n" (at 183.7182 77.724 0)
       (effects (font (size 1.27 1.27)) (justify left))
     )
-    (property "Footprint" "Capacitor_SMD:C_0805_2012Metric" (at 181.5592 91.948 0)
-      (effects (font (size 1.27 1.27)) hide)
-    )
-    (property "Datasheet" "~" (at 180.594 88.138 0)
+    (property "Footprint" "Capacitor_SMD:C_0805_2012Metric" (at 181.5592 80.264 0)
+      (effects (font (size 1.27 1.27)) hide)
+    )
+    (property "Datasheet" "~" (at 180.594 76.454 0)
       (effects (font (size 1.27 1.27)) hide)
     )
@@
     )
   )
-  (symbol (lib_id "Device:C") (at 168.91 88.138 0) (unit 1)
+  (symbol (lib_id "power:VCC") (at 164.592 85.852 0) (unit 1)
+    (in_bom yes) (on_board yes) (dnp no) (fields_autoplaced)
+    (property "Reference" "#PWR013" (at 164.592 89.662 0)
+      (effects (font (size 1.27 1.27)) hide)
+    )
+    (property "Value" "VCC" (at 164.592 81.28 0)
+      (effects (font (size 1.27 1.27)))
+    )
+    (property "Footprint" "" (at 164.592 85.852 0)
+      (effects (font (size 1.27 1.27)) hide)
+    )
+    (property "Datasheet" "" (at 164.592 85.852 0)
+      (effects (font (size 1.27 1.27)) hide)
+    )
+    (pin "1")
+    (instances
+      (project "MCU"
+        (path "/79a91fc1-8991-42e0-8c65-707ff0cecc1c"
+          (reference "#PWR013") (unit 1)
+        )
+      )
+      (project "project233"
+        (path "/a9a55588-2187-4bc3-b43e-c4b5b08bd1ab/543a566d-0d31-4178-abeb-140a350ff13a"
+          (reference "#PWR028") (unit 1)
+        )
+        (path "/a9a55588-2187-4bc3-b43e-c4b5b08bd1ab/c0533110-e4c7-43cb-ae4f-52f25aca33c7"
+          (reference "#PWR037") (unit 1)
+        )
+      )
+      (project "Project232"
+        (path "/b4ba9143-ff4b-4478-b064-00c745ce84f2/ce56912d-0dfe-44d7-8939-923a8b4c6e0e"
+          (reference "#PWR013") (unit 1)
+        )
+      )
+    )
+  )
+  (symbol (lib_id "Device:C") (at 168.91 76.454 0) (unit 1)
     (in_bom yes) (on_board yes) (dnp no)
-    (property "Reference" "C9" (at 172.0342 86.868 0)
+    (property "Reference" "C9" (at 172.0342 75.184 0)
       (effects (font (size 1.27 1.27)) (justify left))
     )
-    (property "Value" "10uF" (at 172.0342 89.408 0)
+    (property "Value" "10uF" (at 172.0342 77.724 0)
       (effects (font (size 1.27 1.27)) (justify left))
     )
-    (property "Footprint" "Capacitor_SMD:C_0805_2012Metric" (at 169.8752 91.948 0)
-      (effects (font (size 1.27 1.27)) hide)
-    )
-    (property "Datasheet" "~" (at 168.91 88.138 0)
+    (property "Footprint" "Capacitor_SMD:C_0805_2012Metric" (at 169.8752 80.264 0)
+      (effects (font (size 1.27 1.27)) hide)
+    )
+    (property "Datasheet" "~" (at 168.91 76.454 0)
       (effects (font (size 1.27 1.27)) hide)
     )
@@
     )
   )
-  (symbol (lib_id "power:+1V8") (at 180.594 81.026 0) (unit 1)
+  (symbol (lib_id "power:+1V8") (at 180.594 69.342 0) (unit 1)
     (in_bom yes) (on_board yes) (dnp no) (fields_autoplaced)
-    (property "Reference" "#PWR023" (at 180.594 84.836 0)
-      (effects (font (size 1.27 1.27)) hide)
-    )
-    (property "Value" "+1V8" (at 180.594 75.692 0)
-      (effects (font (size 1.27 1.27)))
-    )
-    (property "Footprint" "" (at 180.594 81.026 0)
-      (effects (font (size 1.27 1.27)) hide)
-    )
-    (property "Datasheet" "" (at 180.594 81.026 0)
-      (effects (font (size 1.27 1.27)) hide)
-    )
+    (property "Reference" "#PWR023" (at 180.594 73.152 0)
+      (effects (font (size 1.27 1.27)) hide)
+    )
+    (property "Value" "+1V8" (at 180.594 64.008 0)
+      (effects (font (size 1.27 1.27)))
+    )
+    (property "Footprint" "" (at 180.594 69.342 0)
+      (effects (font (size 1.27 1.27)) hide)
+    )
+    (property "Datasheet" "" (at 180.594 69.342 0)
+      (effects (font (size 1.27 1.27)) hide)
+    )

Commit message: update KICAD PCB
Connections:
- net ~INT: now reaches R1.1, U2.13 (~{INT})
Other:
- moved on the sheet: C9, R1
